File: BPS-Minion.sch (KiCad schematic (older format))
At the start: 128 parts, among them J1 TopConn, J10 TempConn2, J2 BottomConn, J3 DTENConfig, J4 IsoConfig, J5 IN, J6 OUT, J8 RegularSPIConn, J9 TempConn1, Q1 BSS308PE, Q10 BSS308PE, Q11 BSS308PE, Q12 BSS308PE, Q13 NSV1C201MZ4, Q2 BSS308PE, Q3 BSS308PE, Q4 BSS308PE, Q5 BSS308PE, Q6 BSS308PE, Q7 BSS308PE, Q8 BSS308PE, Q9 BSS308PE, SW1 Power Switch, U1 LTC6811-1, U2 HX1188FNL, U3 LTC6255, U4 LTC1380, U5 LTC1380

Commit message: Updates HX1188 to point to common library
Parts:
- U2: footprint UTSVT_BPS:HXXXX -> UTSVT_Passive:HXXXX; symbol utsvt-bps:HX1188FNL -> utsvt-chips:HX1188FNL
Changed lines of the file:
@@
 	9550 5050 8250 5050
 $Comp
-L utsvt-bps:HX1188FNL U2
+L utsvt-chips:HX1188FNL U2
 U 1 1 5CAB08B5
 P 10750 1600
 F 0 "U2" H 10750 1765 50  0000 C CNN
 F 1 "HX1188FNL" H 10750 1674 50  0000 C CNN
-F 2 "UTSVT_BPS:HXXXX" H 10750 1600 50  0001 C CNN
+F 2 "UTSVT_Passive:HXXXX" H 10750 1600 50  0001 C CNN
 F 3 "" H 10750 1600 50  0001 C CNN
 	1    10750 1600
