File: BMS.kicad_sch (KiCad schematic)
At the start: 61 parts, among them J1 TopConn, J2 BottomConn, J6 TopConn, U4 BQ7695201PFBR

Commit message: stacked bms schematic
Parts:
- removed C1, C10, C11, C12, C13, C14, C15, C16, C17, C2, C3, C4, C5, C6, C7, C8, C9: 220nF, Capacitor_SMD:C_0805_2012Metric_Pad1.18x1.45mm_HandSolder, symbol Device:C
- removed R1, R10, R11, R12, R13, R14, R15, R16, R17, R2, R3, R4, R5, R6, R7, R8, R9: 20, Resistor_SMD:R_0805_2012Metric_Pad1.20x1.40mm_HandSolder, symbol Device:R_US
- removed TP1, TP10, TP11, TP12, TP13, TP14, TP15, TP2, TP3, TP4, TP5, TP6, TP7, TP8, TP9: TestPoint_2Pole, Jumper:SolderJumper-2_P1.3mm_Open_RoundedPad1.0x1.5mm, symbol Connector:TestPoint_2Pole
- added C1 (x33): 220nF, Capacitor_SMD:C_0805_2012Metric_Pad1.18x1.45mm_HandSolder, symbol Device:C
- added C18: 4.7u, Capacitor_SMD:C_0805_2012Metric_Pad1.18x1.45mm_HandSolder, symbol Device:C
- added C19: 1u, Capacitor_SMD:C_0805_2012Metric_Pad1.18x1.45mm_HandSolder, symbol Device:C
- added C20: 100p, Capacitor_SMD:C_0805_2012Metric_Pad1.18x1.45mm_HandSolder, symbol Device:C
- added C26: .47u, Capacitor_SMD:C_0805_2012Metric_Pad1.18x1.45mm_HandSolder, symbol Device:C
- added D1: BAS16W, Package_TO_SOT_SMD:SOT-323_SC-70, symbol Diode:BAS16W
- added J1, J6: TopConn, Connector_Molex:Molex_Micro-Fit_3.0_43650-0700_1x07_P3.00mm_Horizontal, symbol Connector_Generic:Conn_01x06
- added J10: BMS1OTP, symbol Connector:Conn_01x04_Pin
- added J11: BMS2OTP, symbol Connector:Conn_01x04_Pin
- added J2: BottomConn, Connector_Molex:Molex_Micro-Fit_3.0_43650-0700_1x07_P3.00mm_Horizontal, symbol Connector_Generic:Conn_01x06
- added R1, R10, R11, R12, R13, R14, R15, R16, R2, R3, R4, R5, R58, R59, R6, R60, R61, R62, R63, R64, R65, R66, R67, R68, R69, R7, R70, R71, R72, R73, R74, R8, R9: 20, Resistor_SMD:R_0805_2012Metric, symbol Device:R_Small_US
- added R18, R19: 10k, Resistor_SMD:R_0805_2012Metric_Pad1.20x1.40mm_HandSolder, symbol Device:R_US
- added R20: 100, Resistor_SMD:R_0805_2012Metric_Pad1.20x1.40mm_HandSolder, symbol Device:R_US
- added R77, R78: 10k, Resistor_SMD:R_0805_2012Metric, symbol Device:R_Small_US
- added R79: 100, Resistor_SMD:R_0805_2012Metric, symbol Device:R_Small_US
- added R80: 1k, Resistor_SMD:R_0805_2012Metric, symbol Device:R_Small_US
- added TP15 (x32): TestPoint_2Pole, Jumper:SolderJumper-2_P1.3mm_Open_RoundedPad1.0x1.5mm, symbol Connector:TestPoint_2Pole
- added U10: TCMT1101, Package_SO:SOP-4_4.4x2.6mm_P1.27mm, symbol Isolator:TCMT1101
- added U4: BQ7695201PFBR, Package_QFP:TQFP-48_7x7mm_P0.5mm, symbol utsvt-chips:BQ7695201PFBR
- added U8: ISO1640BDR, Package_SO:SOIC-8_3.9x4.9mm_P1.27mm, symbol utsvt-chips:ISO1640BDR
Connections:
- net GND: now also C1.2, J10.1 (Pin_1), U10.2, U8.4 (GND1); no longer J2.1 (Pin_1)
- net I2C_SCL: now also J10.2 (Pin_2), U8.3 (SCL1)
- net I2C_SDA: now also J10.3 (Pin_3), U8.2 (SDA1)
- net PACK+: now also C1.1, D1.1 (A), J2.3 (Pin_3), R16.1; no longer D1.1 (A), J6.5 (Pin_5), R18.1, R19.1
- net RESET: now also R79.1
- net cell0: now also R58.2, TP15.1
- net cell1: now also R59.2, TP15.1, TP15.2
- net cell10: now also R68.2, TP15.1, TP15.2
- net cell11: now also R69.2, TP15.1, TP15.2
- net cell12: now also R70.2, TP15.1, TP15.2
- net cell13: now also R71.2, TP15.1, TP15.2
- net cell14: now also R72.2, TP15.1, TP15.2
- net cell15: now also R73.2, TP15.1, TP15.2
- net cell16: now also R74.2, TP15.1, TP15.2, U4.16 (VC0)
- net cell2: now also R60.2, TP15.1, TP15.2
- net cell3: now also R61.2, TP15.1, TP15.2
- net cell4: now also R62.2, TP15.1, TP15.2
- net cell5: now also R63.2, TP15.1, TP15.2
- net cell6: now also R64.2, TP15.1, TP15.2
- net cell7: now also R65.2, TP15.1, TP15.2
- net cell8: now also R66.2, TP15.1, TP15.2
- net cell9: now also R67.2, TP15.1, TP15.2
- net at J2.2 (Pin_2): now also C1.1, C1.2, R71.1
- net at J6.3 (Pin_3): now also C1.1, C1.2, R60.1
- net at J2.3 (Pin_3): now also C1.1, C1.2, R72.1
- net at J2.4 (Pin_4): now also C1.1, C1.2, R73.1
- net GND2: now reaches J2.5 (Pin_5)
- net GND2: now also C1.1, C1.2, C18.1, C19.1, C20.1, J11.1 (Pin_1), R74.1, R80.1, U4.17 (VSS), U4.18 (SRP), U4.20 (SRN), U4.36 (REGIN), U4.37 (BREG), U8.5 (GND2)
- net at J2.6 (Pin_6): now also C1.1, C1.2, R1.1
- net at J6.1 (Pin_1): now also C1.1, C1.2, R58.1
- net at J6.2 (Pin_2): now also C1.1, C1.2, R59.1
- net at J6.4 (Pin_4): now also C1.1, C1.2, R61.1
- net at J6.6 (Pin_6): now also C1.1, C1.2, R63.1
- net BMS1BAT: now reaches C19.2, C20.2, C26.2, R20.1, U4.47 (BAT)
- net BMS1BAT: now also J10.4 (Pin_4)
- net at J1.1 (Pin_1): now also C1.1, C1.2, R64.1
- net at J1.2 (Pin_2): now also C1.1, C1.2, R65.1
- net at J1.3 (Pin_3): now also C1.1, C1.2, R66.1
- net at J1.4 (Pin_4): now also C1.1, C1.2, R67.1
- net at J1.5 (Pin_5): now also C1.1, C1.2, R68.1
- net at J1.6 (Pin_6): now also C1.1, C1.2, R69.1
- net BMS1Reg1: now reaches U4.35 (REG1)
- net BMS1Reg1: now also U8.1 (VCC1)
- net FUSE: no longer names the net of U4.38 (FUSE)
- new net: C18.2, U4.24 (REG18)
- new net: C1.1, C1.2, J2.1 (Pin_1), R70.1
- new net: R79.2, U10.1
- new net: C1.1, C1.2, J6.2 (Pin_2), R3.1
- new net: C1.1, C1.2, J1.5 (Pin_5), R12.1
- new net: C1.1, C1.2, J1.3 (Pin_3), R10.1
- new net: C1.1, C1.2, J6.5 (Pin_5), R62.1
- new net: C1.1, C1.2, J6.5 (Pin_5), R6.1
- new net: C1.1, C1.2, J6.4 (Pin_4), R5.1
- new net: C1.1, C1.2, J1.4 (Pin_4), R11.1
- new net: D1.3 (K), R20.2
- new net: C1.1, C1.2, J6.1 (Pin_1), R2.1
- new net: C1.1, C1.2, J6.3 (Pin_3), R4.1
- new net: C1.1, C1.2, J6.6 (Pin_6), R7.1
- new net: C1.1, C1.2, J2.1 (Pin_1), R14.1
- new net: C1.1, C1.2, J1.6 (Pin_6), R13.1
- new net: R19.2, U4.41 (LD)
- new net: R18.2, U4.42 (PACK)
- new net: C26.1, U4.46 (CP1)
- new net: C1.1, C1.2, J1.2 (Pin_2), R9.1
- new net: C1.1, C1.2, J1.1 (Pin_1), R8.1
- new net: C1.1, C1.2, J2.2 (Pin_2), R15.1
- new net BMS2BAT: C19.2, C20.2, C26.2, J11.4 (Pin_4), R20.1, U4.47 (BAT)
- new net BMS2Reg1: R77.1, R78.1, U10.4, U4.35 (REG1), U8.8 (VCC2)
- new net BMS2Reset: R80.2, U10.3, U4.33 (RST_SHUT)
- new net BMS2SCL: J11.2 (Pin_2), R78.2, U4.26 (SCL), U8.6 (SCL2)
- new net BMS2SDA: J11.3 (Pin_3), R77.2, U4.27 (SDA), U8.7 (SDA2)
- new net GND1: D1.1 (A)
- new net PACK1+: R18.1, R18.1, R19.1, R19.1
- new net cell17: R1.2, TP15.1, TP15.2, U4.15 (VC1)
- new net cell18: R2.2, TP15.1, TP15.2, U4.14 (VC2)
- new net cell19: R3.2, TP15.1, TP15.2, U4.13 (VC3)
- new net cell20: R4.2, TP15.1, TP15.2, U4.12 (VC4)
- new net cell21: R5.2, TP15.1, TP15.2, U4.11 (VC5)
- new net cell22: R6.2, TP15.1, TP15.2, U4.10 (VC6)
- new net cell23: R7.2, TP15.1, TP15.2, U4.9 (VC7)
- new net cell24: R8.2, TP15.1, TP15.2, U4.8 (VC8)
- new net cell25: R9.2, TP15.1, TP15.2, U4.7 (VC9)
- new net cell26: R10.2, TP15.1, TP15.2, U4.6 (VC10)
- new net cell27: R11.2, TP15.1, TP15.2, U4.4 (VC12), U4.5 (VC11)
- new net cell28: R12.2, TP15.1, TP15.2, U4.3 (VC13)
- new net cell29: R13.2, TP15.1, TP15.2, U4.2 (VC14)
- new net cell30: R14.2, TP15.1, TP15.2, U4.1 (VC15)
- new net cell31: R15.2, TP15.1, TP15.2, U4.48 (VC16)
- new net cell32: R16.2, TP15.2
- no-connect marks 13 -> 33
Other:
- note added: "BMS1"
- note added: "BMS2"
- note added: "Stack1"
- note added: "Stack2"
- note removed: "BMS"
- moved on the sheet: C18, C19, C20, C26, D1, J1, J2, J6, R18, R19, R20, U4

Commit message: edits to the voltage monitoring board
Parts:
- removed U10: TCMT1101, Package_SO:SOP-4_4.4x2.6mm_P1.27mm, symbol Isolator:TCMT1101
- added R81, R82: 10k, Resistor_SMD:R_0805_2012Metric, symbol Device:R_Small_US
- added R83: 100, Resistor_SMD:R_0805_2012Metric, symbol Device:R_Small_US
- added R84: 1k, Resistor_SMD:R_0805_2012Metric, symbol Device:R_Small_US
- added U10, U12: TLP185, Package_SO:SOIC-4_4.55x3.7mm_P2.54mm, symbol Isolator:TLP185
- added U11: ISO1640BDR, Package_SO:SOIC-8_3.9x4.9mm_P1.27mm, symbol utsvt-chips:ISO1640BDR
- J10, J11: footprint (none) -> Connector_PinHeader_2.54mm:PinHeader_1x04_P2.54mm_Vertical
Connections:
- net BMS1Reg1: now also R81.1, R82.1, U10.6, U11.8 (VCC2); no longer U8.1 (VCC1)
- net BMS2Reg1: now also U12.6
- net BMS2Reset: now also U12.4
- net GND: now also U10.3, U12.3; no longer C1.2, C18.1, C19.1, C20.1, J10.1 (Pin_1), U4.17 (VSS), U4.18 (SRP), U4.20 (SRN), U4.36 (REGIN), U4.37 (BREG), U8.4 (GND1)
- net GND1: now also C1.2, C18.1, C19.1, C20.1, J10.1 (Pin_1), U4.17 (VSS), U4.18 (SRP), U4.20 (SRN), U4.36 (REGIN), U4.37 (BREG), U8.4 (GND1), R84.1, U11.4 (GND1); no longer D1.1 (A)
- net GND2: now also D1.1 (A), U11.5 (GND2)
- net I2C_SCL: now also U11.3 (SCL1); no longer U4.26 (SCL)
- net I2C_SDA: now also U11.2 (SDA1); no longer U4.27 (SDA)
- net RESET: now also R83.1; no longer U4.33 (RST_SHUT)
- net at R79.2: now also U12.1
- new net: R83.2, U10.1
- new net +3.3V: U11.1 (VCC1), U8.1 (VCC1)
- new net BMS1Reset: R84.2, U10.4, U4.33 (RST_SHUT)
- new net BMS1SCL: R82.2, U11.6 (SCL2), U4.26 (SCL)
- new net BMS1SDA: R81.2, U11.7 (SDA2), U4.27 (SDA)
Other:
- moved on the sheet: C1, C18, C19, C20, C26, D1, J1, J10, J11, J2, J6, R1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

Commit message: final edits
Parts:
- R79, R83: value 100 -> 220
Connections:
- net GND: now also U11.4 (GND1), U8.4 (GND1)
- net GND1: now also U11.5 (GND2); no longer U11.4 (GND1), U8.4 (GND1)
- net GND2: now also R18.1, R19.1; no longer U11.5 (GND2)
- net PACK1+: no longer R18.1, R19.1
Changed lines of the file:
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@@
   (junction (at 167.64 220.98) (diameter 0) (color 0 0 0 0)
   )
+  (junction (at 92.71 46.355) (diameter 0) (color 0 0 0 0)
+  )
   (junction (at 289.56 207.01) (diameter 0) (color 0 0 0 0)
   )
@@
     (stroke (width 0) (type default))
   )
+  (wire (pts (xy 92.71 46.355) (xy 92.71 48.895))
+    (stroke (width 0) (type default))
+  )
   (wire (pts (xy 191.77 184.785) (xy 191.77 189.23))
     (stroke (width 0) (type default))
@@
     (stroke (width 0) (type default))
   )
+  (wire (pts (xy 92.71 46.355) (xy 95.25 46.355))
+    (stroke (width 0) (type default))
+  )
   (wire (pts (xy 66.04 207.01) (xy 67.31 207.01))
     (stroke (width 0) (type default))
@@
     (effects (font (size 1.27 1.27)) (justify left bottom))
   )
-  (label "PACK1+" (at 92.71 48.895 0) (fields_autoplaced)
-    (effects (font (size 1.27 1.27)) (justify left bottom))
-  )
   (label "cell3" (at 76.2 224.79 270) (fields_autoplaced)
     (effects (font (size 1.27 1.27)) (justify right bottom))
@@
     (effects (font (size 1.27 1.27)) (justify right bottom))
   )
-  (label "PACK1+" (at 92.71 46.355 0) (fields_autoplaced)
-    (effects (font (size 1.27 1.27)) (justify left bottom))
-  )
   (label "BMS2BAT" (at 344.805 28.575 180) (fields_autoplaced)
     (effects (font (size 1.27 1.27)) (justify right bottom))
@@
       (effects (font (size 1.27 1.27)))
     )
-    (property "Value" "100" (at 333.375 139.065 90)
+    (property "Value" "220" (at 333.375 139.065 90)
       (effects (font (size 1.27 1.27)))
     )
@@
       (effects (font (size 1.27 1.27)))
     )
-    (property "Value" "100" (at 74.93 101.6 90)
+    (property "Value" "220" (at 74.93 101.6 90)
       (effects (font (size 1.27 1.27)))
     )
@@
     )
   )
+  (symbol (lib_id "power:GND1") (at 86.36 144.145 0) (unit 1)
+    (in_bom yes) (on_board yes) (dnp no) (fields_autoplaced)
+    (property "Reference" "#PWR078" (at 86.36 150.495 0)
+      (effects (font (size 1.27 1.27)) hide)
+    )
+    (property "Value" "GND1" (at 86.36 149.225 0)
+      (effects (font (size 1.27 1.27)))
+    )
+    (property "Footprint" "" (at 86.36 144.145 0)
+      (effects (font (size 1.27 1.27)) hide)
+    )
+    (property "Datasheet" "" (at 86.36 144.145 0)
+      (effects (font (size 1.27 1.27)) hide)
+    )
+    (pin "1")
+    (instances
+      (project "BPS-Minion"
+        (path "/86f4c077-2357-4bc0-9102-0d9b954ffb24/f4179d79-1229-45f6-9801-99c07e86bfe4"
+          (reference "#PWR078") (unit 1)
+        )
+      )
+    )
+  )
   (symbol (lib_id "Connector:TestPoint_2Pole") (at 71.12 220.98 0) (unit 1)
     (in_bom yes) (on_board yes) (dnp no)
@@
     )
   )
-  (symbol (lib_id "power:GND1") (at 45.72 144.145 0) (unit 1)
-    (in_bom yes) (on_board yes) (dnp no) (fields_autoplaced)
-    (property "Reference" "#PWR074" (at 45.72 150.495 0)
-      (effects (font (size 1.27 1.27)) hide)
-    )
-    (property "Value" "GND1" (at 45.72 149.225 0)
-      (effects (font (size 1.27 1.27)))
-    )
-    (property "Footprint" "" (at 45.72 144.145 0)
-      (effects (font (size 1.27 1.27)) hide)
-    )
-    (property "Datasheet" "" (at 45.72 144.145 0)
-      (effects (font (size 1.27 1.27)) hide)
-    )
-    (pin "1")
-    (instances
-      (project "BPS-Minion"
-        (path "/86f4c077-2357-4bc0-9102-0d9b954ffb24/f4179d79-1229-45f6-9801-99c07e86bfe4"
-          (reference "#PWR074") (unit 1)
-        )
-      )
-    )
-  )
   (symbol (lib_id "Connector:TestPoint_2Pole") (at 111.76 220.98 0) (unit 1)
     (in_bom yes) (on_board yes) (dnp no)
@@
     )
   )
-  (symbol (lib_id "power:GND1") (at 318.77 119.38 0) (unit 1)
+  (symbol (lib_id "power:GND2") (at 95.25 46.355 0) (unit 1)
     (in_bom yes) (on_board yes) (dnp no) (fields_autoplaced)
-    (property "Reference" "#PWR067" (at 318.77 125.73 0)
+    (property "Reference" "#PWR074" (at 95.25 52.705 0)
       (effects (font (size 1.27 1.27)) hide)
     )
-    (property "Value" "GND1" (at 318.77 124.46 0)
+    (property "Value" "GND2" (at 95.25 50.8 0)
       (effects (font (size 1.27 1.27)))
     )
-    (property "Footprint" "" (at 318.77 119.38 0)
+    (property "Footprint" "" (at 95.25 46.355 0)
       (effects (font (size 1.27 1.27)) hide)
     )
-    (property "Datasheet" "" (at 318.77 119.38 0)
+    (property "Datasheet" "" (at 95.25 46.355 0)
       (effects (font (size 1.27 1.27)) hide)
     )
@@
       (project "BPS-Minion"
         (path "/86f4c077-2357-4bc0-9102-0d9b954ffb24/f4179d79-1229-45f6-9801-99c07e86bfe4"
-          (reference "#PWR067") (unit 1)
+          (reference "#PWR074") (unit 1)
         )
       )
@@
     )
   )
+  (symbol (lib_id "power:GND") (at 45.72 144.145 0) (unit 1)
+    (in_bom yes) (on_board yes) (dnp no) (fields_autoplaced)
+    (property "Reference" "#PWR075" (at 45.72 150.495 0)
+      (effects (font (size 1.27 1.27)) hide)
+    )
+    (property "Value" "GND" (at 45.72 149.225 0)
+      (effects (font (size 1.27 1.27)))
+    )
+    (property "Footprint" "" (at 45.72 144.145 0)
+      (effects (font (size 1.27 1.27)) hide)
+    )
+    (property "Datasheet" "" (at 45.72 144.145 0)
+      (effects (font (size 1.27 1.27)) hide)
+    )
+    (pin "1")
+    (instances
+      (project "BPS-Minion"
+        (path "/86f4c077-2357-4bc0-9102-0d9b954ffb24/f4179d79-1229-45f6-9801-99c07e86bfe4"
+          (reference "#PWR075") (unit 1)
+        )
+      )
+    )
+  )
   (symbol (lib_id "power:GND1") (at 31.75 106.045 0) (unit 1)
     (in_bom yes) (on_board yes) (dnp no) (fields_autoplaced)
@@
     )
   )
-  (symbol (lib_id "power:GND2") (at 86.36 144.145 0) (unit 1)
-    (in_bom yes) (on_board yes) (dnp no) (fields_autoplaced)
-    (property "Reference" "#PWR075" (at 86.36 150.495 0)
-      (effects (font (size 1.27 1.27)) hide)
-    )
-    (property "Value" "GND2" (at 86.36 148.59 0)
-      (effects (font (size 1.27 1.27)))
-    )
-    (property "Footprint" "" (at 86.36 144.145 0)
-      (effects (font (size 1.27 1.27)) hide)
-    )
-    (property "Datasheet" "" (at 86.36 144.145 0)
-      (effects (font (size 1.27 1.27)) hide)
-    )
-    (pin "1")
-    (instances
-      (project "BPS-Minion"
-        (path "/86f4c077-2357-4bc0-9102-0d9b954ffb24/f4179d79-1229-45f6-9801-99c07e86bfe4"
-          (reference "#PWR075") (unit 1)
-        )
-      )
-    )
-  )
   (symbol (lib_id "Device:R_Small_US") (at 358.14 151.765 180) (unit 1)
     (in_bom yes) (on_board yes) (dnp no) (fields_autoplaced)
@@
         )
       )
+    )
+  )
+  (symbol (lib_id "power:GND") (at 318.77 119.38 0) (unit 1)
+    (in_bom yes) (on_board yes) (dnp no) (fields_autoplaced)
+    (property "Reference" "#PWR067" (at 318.77 125.73 0)
+      (effects (font (size 1.27 1.27)) hide)
+    )
+    (property "Value" "GND" (at 318.77 124.46 0)
+      (effects (font (size 1.27 1.27)))
+    )
+    (property "Footprint" "" (at 318.77 119.38 0)
+      (effects (font (size 1.27 1.27)) hide)
+    )
+    (property "Datasheet" "" (at 318.77 119.38 0)
+      (effects (font (size 1.27 1.27)) hide)
+    )
+    (pin "1")
+    (instances
+      (project "BPS-Minion"
+        (path "/86f4c077-2357-4bc0-9102-0d9b954ffb24/f4179d79-1229-45f6-9801-99c07e86bfe4"
+          (reference "#PWR067") (unit 1)
+        )
+      )
