File: BPS-Minion.kicad_pcb (KiCad board)
At the start: 2 copper layers, 85 x 128 mm, 219 parts, among them J10 TopConn, J11 TopConn, J2 BMS1OTP, J3 BMS2OTP, J4 Conn_01x24_Female, J5 Conn_01x24_Female, J6 TopConn, J7 TopConn, J8 TopConn, J9 TopConn, U10 LM321, U11 ADS7953SBDBT, U12 MIC5317-2.5xM5, U2 BQ7695201PFBR, U3 ISO1640BDR, U4 EL3H7, U5 BQ7695201PFBR, U6 ISO1640BDR, U7 EL3H7, U8 LM321, U9 ADS7953SBDBT

Commit message: submodule fixes and updte PCB
Parts:
- moved R92 249.6 mm to (153.2, 195.3)
- moved D3 0.89 mm to (58.9, 67.1)
Changed lines of the file:
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@@
   )
   (footprint "Diode_SMD:D_SOD-123" (layer "F.Cu")
-    (at 58.554 66.247)
+    (at 58.926 67.056)
     (descr "SOD-123")
     (tags "SOD-123")
@@
   )
   (footprint "Resistor_SMD:R_0805_2012Metric" (layer "F.Cu")
-    (at -60.6232 66.4816)
+    (at 153.16 195.326)
     (descr "Resistor SMD 0805 (2012 Metric), square (rectangular) end terminal, IPC_7351 nominal, (Body size source: IPC-SM-782 page 72, https://www.pcb-3d.com/wordpress/wp-content/uploads/ipc-sm-782a_amendment_1_and_2.pdf), generated with kicad-footprint-generator")
     (tags "resistor")
@@
     (property "Sheetfile" "Temperature.kicad_sch")
     (property "Sheetname" "Temperature1")
-    (property "ki_description" "Generic connector, single row, 01x24, script generated (kicad-library-utils/schlib/autogen/connector/)")
+    (property "ki_description" "Generic connector, single row, 01x24, script generated")
     (property "ki_keywords" "connector")
     (attr through_hole)
@@
     (property "Sheetfile" "Temperature.kicad_sch")
     (property "Sheetname" "Temperature")
-    (property "ki_description" "Generic connector, single row, 01x24, script generated (kicad-library-utils/schlib/autogen/connector/)")
+    (property "ki_description" "Generic connector, single row, 01x24, script generated")
     (property "ki_keywords" "connector")
     (attr through_hole)

Commit message: started layout
Parts:
- C15, C16, C17, C18, C19, C61, R17, R18, R19, R20, R21, R22, R23, R24, R25, R26, R27, R28, R29, R30, R31, R32, R33, R34, R89, R91, U8: moved to B.Cu
- moved MH3 246.5 mm to (51.9, 175.6)
- moved J11 232.1 mm to (123.7, 152.9), turned to -90 degrees
- moved R83 231.3 mm to (115.3, 155.1), turned to 180 degrees
- moved R84 230.7 mm to (115.3, 157.4), turned to 180 degrees
- moved R85 230.0 mm to (115.3, 159.6), turned to 180 degrees
- moved C55 229.9 mm to (112.3, 153.8), turned to 90 degrees
- moved C56 229.5 mm to (108.7, 156.1), turned to 90 degrees
- moved R86 229.4 mm to (115.3, 161.9), turned to 180 degrees
- moved R87 228.7 mm to (115.3, 164.2), turned to 180 degrees
- moved C57 228.5 mm to (112.3, 158.4), turned to 90 degrees
- moved TP36 228.2 mm to (103.7, 169.8), turned to -90 degrees
- moved R88 228.0 mm to (115.3, 166.5), turned to 180 degrees
- moved C58 228.0 mm to (108.7, 160.7), turned to 90 degrees
- moved MH1 228.0 mm to (51.9, 30.1)
- moved TP35 228.0 mm to (103.7, 166.0), turned to -90 degrees
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Routing:
- net /BMS/cell15: track 0.00 -> 56.7 mm
- net /Temperature/temp9: track 0.00 -> 53.2 mm
- net /BMS/cell14: track 0.00 -> 52.2 mm
- net /Temperature/temp10: track 0.00 -> 49.6 mm
- net /Temperature/temp3: track 0.00 -> 49.3 mm
- net /BMS/cell11: track 0.00 -> 49.3 mm
- net /BMS/cell13: track 0.00 -> 48.8 mm
- net /BMS/cell12: track 0.00 -> 45.6 mm
- net /Temperature/temp4: track 0.00 -> 44.5 mm
- net /Temperature/temp11: track 0.00 -> 44.2 mm
- net /Temperature/temp12: track 0.00 -> 40.4 mm
- net /Temperature/temp5: track 0.00 -> 38.2 mm
- net /Temperature/temp13: track 0.00 -> 36.8 mm
- net /BMS/cell10: track 0.00 -> 36.4 mm
- net /Temperature/temp6: track 0.00 -> 34.6 mm
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Other:
- board size 85 x 128 mm -> 85 x 152 mm
- board text added: "Grid size is .2540 mm"

Commit message: minor temp changes
Parts:
- moved C61 5.75 mm to (72.6, 51.6)
- moved C18 4.06 mm to (72.6, 49.5)
- moved R34 3.40 mm to (65.5, 52.1), turned to -90 degrees
- moved C19 3.06 mm to (68.6, 55.9), turned to 180 degrees
- moved C17 1.02 mm to (63.8, 52.1)
- moved U8 0.88 mm to (60.6, 52.1)
Routing:
- net /BMS/cell0: track 35.0 -> 37.5 mm
Changed lines of the file:
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@@
   )
   (footprint "Resistor_SMD:R_0805_2012Metric_Pad1.20x1.40mm_HandSolder" (layer "B.Cu")
-    (at 63.992 49.022)
+    (at 65.532 52.054 -90)
     (descr "Resistor SMD 0805 (2012 Metric), square (rectangular) end terminal, IPC_7351 nominal with elongated pad for handsoldering. (Body size source: IPC-SM-782 page 72, https://www.pcb-3d.com/wordpress/wp-content/uploads/ipc-sm-782a_amendment_1_and_2.pdf), generated with kicad-footprint-generator")
     (tags "resistor handsolder")
@@
     (property "ki_keywords" "R res resistor")
     (attr smd)
-    (fp_text reference "R34" (at 0 1.65) (layer "B.SilkS")
-        (effects (font (size 1 1) (thickness 0.15)) (justify mirror))
-    )
-    (fp_text value "4.7k" (at 0 -1.65) (layer "B.Fab")
-        (effects (font (size 1 1) (thickness 0.15)) (justify mirror))
-    )
-    (fp_text user "${REFERENCE}" (at 0 0) (layer "B.Fab")
+    (fp_text reference "R34" (at 0 1.65 90) (layer "B.SilkS")
+        (effects (font (size 1 1) (thickness 0.15)) (justify mirror))
+    )
+    (fp_text value "4.7k" (at 0 -1.65 90) (layer "B.Fab")
+        (effects (font (size 1 1) (thickness 0.15)) (justify mirror))
+    )
+    (fp_text user "${REFERENCE}" (at 0 0 90) (layer "B.Fab")
         (effects (font (size 0.5 0.5) (thickness 0.08)) (justify mirror))
     )
@@
     (fp_line (start 1 0.625) (end 1 -0.625)
       (stroke (width 0.1) (type solid)) (layer "B.Fab"))
-    (pad "1" smd roundrect (at -1 0) (size 1.2 1.4) (layers "B.Cu" "B.Paste" "B.Mask") (roundrect_rratio 0.208333)
+    (pad "1" smd roundrect (at -1 0 270) (size 1.2 1.4) (layers "B.Cu" "B.Paste" "B.Mask") (roundrect_rratio 0.208333)
       (net 22 "Net-(U8-+)") (pintype "passive"))
-    (pad "2" smd roundrect (at 1 0) (size 1.2 1.4) (layers "B.Cu" "B.Paste" "B.Mask") (roundrect_rratio 0.208333)
+    (pad "2" smd roundrect (at 1 0 270) (size 1.2 1.4) (layers "B.Cu" "B.Paste" "B.Mask") (roundrect_rratio 0.208333)
       (net 202 "Net-(C16-Pad2)") (pintype "passive"))
     (model "${KICAD6_3DMODEL_DIR}/Resistor_SMD.3dshapes/R_0805_2012Metric.wrl"
@@
   )
   (footprint "Package_TO_SOT_SMD:SOT-23-5" (layer "B.Cu")
-    (at 61.468 52.07 180)
+    (at 60.5845 52.07 180)
     (descr "SOT, 5 Pin (https://www.jedec.org/sites/default/files/docs/Mo-178c.PDF variant AA), generated with kicad-footprint-generator ipc_gullwing_generator.py")
     (tags "SOT TO_SOT_SMD")
@@
   )
   (footprint "Capacitor_SMD:C_0805_2012Metric_Pad1.18x1.45mm_HandSolder" (layer "B.Cu")
-    (at 64.77 52.07 90)
+    (at 63.754 52.07 90)
     (descr "Capacitor SMD 0805 (2012 Metric), square (rectangular) end terminal, IPC_7351 nominal with elongated pad for handsoldering. (Body size source: IPC-SM-782 page 76, https://www.pcb-3d.com/wordpress/wp-content/uploads/ipc-sm-782a_amendment_1_and_2.pdf, https://docs.google.com/spreadsheets/d/1BsfQQcO9C6DZCsRaXUlFlo91Tg2WpOkGARC1WS5S8t0/edit?usp=sharing), generated with kicad-footprint-generator")
     (tags "capacitor handsolder")
@@
   )
   (footprint "Capacitor_SMD:C_0805_2012Metric_Pad1.18x1.45mm_HandSolder" (layer "B.Cu")
-    (at 68.58 55.626)
+    (at 72.644 51.562)
     (descr "Capacitor SMD 0805 (2012 Metric), square (rectangular) end terminal, IPC_7351 nominal with elongated pad for handsoldering. (Body size source: IPC-SM-782 page 76, https://www.pcb-3d.com/wordpress/wp-content/uploads/ipc-sm-782a_amendment_1_and_2.pdf, https://docs.google.com/spreadsheets/d/1BsfQQcO9C6DZCsRaXUlFlo91Tg2WpOkGARC1WS5S8t0/edit?usp=sharing), generated with kicad-footprint-generator")
     (tags "capacitor handsolder")
@@
   )
   (footprint "Capacitor_SMD:C_0805_2012Metric_Pad1.18x1.45mm_HandSolder" (layer "B.Cu")
-    (at 65.532 56.1125 -90)
+    (at 68.58 55.88 180)
     (descr "Capacitor SMD 0805 (2012 Metric), square (rectangular) end terminal, IPC_7351 nominal with elongated pad for handsoldering. (Body size source: IPC-SM-782 page 76, https://www.pcb-3d.com/wordpress/wp-content/uploads/ipc-sm-782a_amendment_1_and_2.pdf, https://docs.google.com/spreadsheets/d/1BsfQQcO9C6DZCsRaXUlFlo91Tg2WpOkGARC1WS5S8t0/edit?usp=sharing), generated with kicad-footprint-generator")
     (tags "capacitor handsolder")
@@
     (property "ki_keywords" "cap capacitor")
     (attr smd)
-    (fp_text reference "C19" (at 0 1.68 90) (layer "B.SilkS")
-        (effects (font (size 1 1) (thickness 0.15)) (justify mirror))
-    )
-    (fp_text value "1u" (at 0 -1.68 90) (layer "B.Fab")
-        (effects (font (size 1 1) (thickness 0.15)) (justify mirror))
-    )
-    (fp_text user "${REFERENCE}" (at 0 0 90) (layer "B.Fab")
+    (fp_text reference "C19" (at 0 1.68) (layer "B.SilkS")
+        (effects (font (size 1 1) (thickness 0.15)) (justify mirror))
+    )
+    (fp_text value "1u" (at 0 -1.68) (layer "B.Fab")
+        (effects (font (size 1 1) (thickness 0.15)) (justify mirror))
+    )
+    (fp_text user "${REFERENCE}" (at 0 0) (layer "B.Fab")
         (effects (font (size 0.5 0.5) (thickness 0.08)) (justify mirror))
     )
@@
     (fp_line (start 1 0.625) (end 1 -0.625)
       (stroke (width 0.1) (type solid)) (layer "B.Fab"))
-    (pad "1" smd roundrect (at -1.0375 0 270) (size 1.175 1.45) (layers "B.Cu" "B.Paste" "B.Mask") (roundrect_rratio 0.212766)
+    (pad "1" smd roundrect (at -1.0375 0 180) (size 1.175 1.45) (layers "B.Cu" "B.Paste" "B.Mask") (roundrect_rratio 0.212766)
       (net 24 "VDDA") (pintype "passive"))
-    (pad "2" smd roundrect (at 1.0375 0 270) (size 1.175 1.45) (layers "B.Cu" "B.Paste" "B.Mask") (roundrect_rratio 0.212766)
+    (pad "2" smd roundrect (at 1.0375 0 180) (size 1.175 1.45) (layers "B.Cu" "B.Paste" "B.Mask") (roundrect_rratio 0.212766)
       (net 23 "GNDA") (pintype "passive"))
     (model "${KICAD6_3DMODEL_DIR}/Capacitor_SMD.3dshapes/C_0805_2012Metric.wrl"
@@
   )
   (footprint "Capacitor_SMD:C_0805_2012Metric_Pad1.18x1.45mm_HandSolder" (layer "B.Cu")
-    (at 72.644 45.466 180)
+    (at 72.644 49.53 180)
     (descr "Capacitor SMD 0805 (2012 Metric), square (rectangular) end terminal, IPC_7351 nominal with elongated pad for handsoldering. (Body size source: IPC-SM-782 page 76, https://www.pcb-3d.com/wordpress/wp-content/uploads/ipc-sm-782a_amendment_1_and_2.pdf, https://docs.google.com/spreadsheets/d/1BsfQQcO9C6DZCsRaXUlFlo91Tg2WpOkGARC1WS5S8t0/edit?usp=sharing), generated with kicad-footprint-generator")
     (tags "capacitor handsolder")
@@
   (segment (start 103.666 38.633767) (end 107.8635 38.633767) (width 0.2) (layer "F.Cu") (net 127))
   (segment (start 103.291736 38.633767) (end 102.616 39.309503) (width 0.2) (layer "F.Cu") (net 127))
+  (segment (start 103.666 36.123767) (end 103.666 38.633767) (width 0.2) (layer "F.Cu") (net 127))
   (segment (start 102.216 49.754131) (end 94.9095 57.060631) (width 0.2) (layer "F.Cu") (net 128))
   (segment (start 103.666 42.443767) (end 107.8935 42.443767) (width 0.2) (layer "F.Cu") (net 128))

Commit message: new temp layout (bottom one)
Parts:
- R35, R36, R37, R38, R39, R40, R41, R42, R43, R44, R45, R46, R47, R48, R49, R50: moved to B.Cu
- moved C20 176.7 mm to (86.6, 159.5)
- moved C23 171.3 mm to (83.6, 148.8)
- moved C24 171.0 mm to (82.5, 159.5)
- moved C62 171.0 mm to (83.6, 146.8), turned to 180 degrees
- moved R36 148.4 mm to (62.8, 160.5)
- moved R38 147.0 mm to (62.8, 158.4)
- moved R39 145.2 mm to (62.8, 162.5)
- moved J5 144.9 mm to (57.3, 166.3)
- moved R41 144.3 mm to (62.8, 164.5)
- moved R40 142.8 mm to (62.6, 154.4)
- moved R43 141.9 mm to (62.8, 166.6)
- moved R42 141.8 mm to (62.6, 152.3)
- moved U11 140.4 mm to (80.6, 153.9), turned to -90 degrees
- moved R35 139.9 mm to (54.0, 158.2), turned to 180 degrees
- moved R37 139.2 mm to (54.0, 160.2), turned to 180 degrees
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Routing:
- net /Temperature1/temp1: track 0.00 -> 68.3 mm, vias 0 -> 3
- net /Temperature1/temp2: track 0.00 -> 62.5 mm, vias 0 -> 3
- net /Temperature1/temp8: track 0.00 -> 55.2 mm, vias 0 -> 3
- net /Temperature1/temp7: track 0.00 -> 50.6 mm, vias 0 -> 3
- net /Temperature1/temp6: track 0.00 -> 38.9 mm, vias 0 -> 1
- net /Temperature1/temp16: track 0.00 -> 36.1 mm, vias 0 -> 1
- net /Temperature1/temp5: track 0.00 -> 30.0 mm, vias 0 -> 1
- net /Temperature1/temp4: track 0.00 -> 28.7 mm, vias 0 -> 1
- net /Temperature1/temp3: track 0.00 -> 26.8 mm, vias 0 -> 1
- net /Temperature1/temp15: track 0.00 -> 26.2 mm, vias 0 -> 1
- net /Temperature1/temp9: track 0.00 -> 24.9 mm, vias 0 -> 1
- net /Temperature1/temp10: track 0.00 -> 24.7 mm, vias 0 -> 1
- net /Temperature1/temp14: track 0.00 -> 23.8 mm, vias 0 -> 1
- net /Temperature1/temp13: track 0.00 -> 22.9 mm, vias 0 -> 1
- net /Temperature1/temp12: track 0.00 -> 22.3 mm, vias 0 -> 1
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
Commit message: time flies when you're kicadding :(
Parts:
- C1, C10, C11, C12, C13, C14, C15, C16, C17, C18, C19, C2, C20, C21, C22, C23, C24, C25, C26, C27, C28, C29, C3, C30, C31, C32, C33, C34, C35, C36, C37, C38, C39, C4, C40, C41, C42, C43, C44, C45, C46, C47, C48, C49, C5, C50, C51, C52, C53, C54, C55, C56, C57, C58, C59, C6, C60, C61, C62, C7, C8, C9: footprint Capacitor_SMD:C_0805_2012Metric_Pad1.18x1.45mm_HandSolder -> Capacitor_SMD:C_0805_2012Metric
- R11, R12, R16, R33, R34, R5, R51, R52, R6, R89, R9, R90, R91, R94: footprint Resistor_SMD:R_0805_2012Metric_Pad1.20x1.40mm_HandSolder -> Resistor_SMD:R_0805_2012Metric
- R13: footprint Resistor_SMD:R_0805_2012Metric -> Resistor_SMD:R_0805_2012Metric_Pad1.20x1.40mm_HandSolder
- moved C18 83.0 mm to (-10.3, 45.9)
- moved C61 83.0 mm to (-10.3, 48.0)
- moved R33 83.0 mm to (-14.3, 48.0)
- moved U9 83.0 mm to (-11.0, 47.1)
- moved C15 83.0 mm to (-14.3, 41.9)
- moved C16 83.0 mm to (-14.3, 45.9)
- moved C17 83.0 mm to (-19.2, 48.5)
- moved C19 83.0 mm to (-14.3, 52.3)
- moved R17 83.0 mm to (-22.5, 43.1)
- moved R18 83.0 mm to (-31.2, 41.0)
- moved R19 83.0 mm to (-22.5, 41.0)
- moved R20 83.0 mm to (-31.2, 43.1)
- moved R21 83.0 mm to (-31.2, 39.0)
- moved R22 83.0 mm to (-31.2, 46.9)
- moved R23 83.0 mm to (-31.2, 37.0)
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Routing:
- net /BMS/BMS1BAT: track 0.00 -> 20.6 mm
- net /BMS/BMS1SDA: track 0.00 -> 19.6 mm, vias 0 -> 1
- net /BMS/BMS1SCL: track 0.00 -> 19.6 mm, vias 0 -> 1
- net /BMS/BMS1Reg1: track 0.00 -> 13.5 mm
- net Net-(U2-LD): track 0.00 -> 11.1 mm
- net Net-(U2-PACK): track 0.00 -> 9.69 mm
- net Net-(U2-CP1): track 0.05 -> 9.68 mm
- net Net-(D2-K): track 0.00 -> 7.68 mm
- net Net-(J9-Pin_4): track 12.5 -> 5.61 mm
- net Net-(J10-Pin_4): track 12.5 -> 5.61 mm
- net Net-(J6-Pin_4): track 12.5 -> 5.61 mm
- net Net-(J8-Pin_4): track 12.5 -> 5.61 mm
- net Net-(J7-Pin_4): track 12.5 -> 5.61 mm
- net Net-(J11-Pin_4): track 12.5 -> 5.61 mm
- net /BMS/cell1: track 31.6 -> 38.2 mm
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
Commit message: wheeeeeee
Parts:
- moved R3 25.2 mm to (91.7, 75.9), turned to 0 degrees
- moved U4 21.4 mm to (91.7, 69.8), turned to 90 degrees
- moved J2 14.5 mm to (85.8, 49.3), turned to -90 degrees
- moved R7 9.43 mm to (81.8, 69.6), turned to 0 degrees
- moved R92 8.94 mm to (74.3, 112.8)
- moved C8 7.37 mm to (77.0, 69.6)
- moved C6 7.37 mm to (77.0, 71.9)
- moved R9 7.37 mm to (77.0, 67.3), turned to 0 degrees
- moved C7 5.09 mm to (77.0, 55.9)
- moved C5 5.09 mm to (77.0, 62.7)
- moved R5 5.09 mm to (77.0, 60.5)
- moved R6 5.09 mm to (77.0, 58.2)
- moved R8 5.09 mm to (77.0, 53.6)
- moved C4 4.52 mm to (90.4, 52.1), turned to 135 degrees
- moved D2 1.80 mm to (76.5, 65.0)
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Routing:
- net GND2: track 14.6 -> 84.5 mm
- net GND1: track 9.63 -> 38.9 mm, vias 0 -> 6
- net /BMS/BMS1Reg1: track 13.5 -> 30.4 mm, vias 0 -> 2
- net /BMS/BMS1Reset: track 5.28 -> 21.8 mm, vias 0 -> 2
- net /BMS/BMS1BAT: track 20.6 -> 34.4 mm, vias 0 -> 2
- net /BMS/BMS1SCL: track 19.6 -> 25.3 mm, vias 1 -> 2
- net /BMS/BMS1SDA: track 19.6 -> 25.2 mm, vias 1 -> 2
- net Net-(D2-K): track 7.68 -> 2.72 mm, vias 0 -> 2
- net Net-(U2-LD): track 11.1 -> 6.50 mm
- net Net-(U2-PACK): track 9.69 -> 6.09 mm
- net Net-(R3-Pad2): track 0.00 -> 3.55 mm
- net Net-(U2-REG18): track 0.00 -> 3.02 mm
- net Net-(U2-CP1): track 9.68 -> 7.15 mm
- net +3.3V: track 2.99 -> 2.00 mm
- added copper zone on B.Cu, net GND1
- added copper zone on F.Cu, net GND1
Other:
- board text removed: "MH1"
- board text removed: "MH2"
- board text removed: "Peripheral SOM"
