File: BPS-Minion.kicad_sch (KiCad schematic)
At the start: 11 parts, among them U12 MIC5317-2.5xM5

Commit message: wheeeeeee
Other:
- moved on the sheet: D1, R1, R92

Commit message: literal piss and shit
Parts:
- C1: value 10u -> 10uF
- C2: value 1u -> 1uF
- R1: footprint Resistor_SMD:R_0805_2012Metric_Pad1.20x1.40mm_HandSolder -> Resistor_SMD:R_0805_2012Metric
Changed lines of the file:
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@@
       (effects (font (size 1.27 1.27)) (justify right))
     )
-    (property "Value" "1u" (at 230.505 104.775 0)
+    (property "Value" "1uF" (at 230.505 104.775 0)
       (effects (font (size 1.27 1.27)) (justify right))
     )
@@
       (effects (font (size 1.27 1.27)))
     )
-    (property "Footprint" "Resistor_SMD:R_0805_2012Metric_Pad1.20x1.40mm_HandSolder" (at 168.529 48.006 90)
+    (property "Footprint" "Resistor_SMD:R_0805_2012Metric" (at 168.529 48.006 90)
       (effects (font (size 1.27 1.27)) hide)
     )
@@
       (effects (font (size 1.27 1.27)) (justify right))
     )
-    (property "Value" "10u" (at 192.405 107.95 0)
-      (effects (font (size 1.27 1.27)) (justify right))
-    )
+    (property "Value" "10uF" (at 192.405 107.95 0)
+      (effects (font (size 1.27 1.27)) (justify right))
+    )
